Commit message: Use xacro to generate urdf.

File: chapter6_ws/src/firstbot_description/urdf/first_robot.xacro (robot description, xacro)
@@ -1,32 +1,38 @@
 <?xml version="1.0"?>
-<robot name="first_robot">
-  <!-- Robot Body -->
-  <link name="base_link">
-    <!-- Appearance -->
-    <visual>
-      <origin xyz="0.0 0.0 0.0" rpy="0.0 0.0 0.0" />
-      <geometry>
-        <cylinder radius="0.1" length="0.12"/>
-      </geometry>
-      <material name="white">
-        <color rgba="1.0 1.0 1.0 0.5"/>
+<robot xmlns:xacro="http://www.ros.org/wiki/xacro" name="first_robot">
+  <xacro:macro name="base_link" params="radius length">
+    <link name="base_link">
+      <!-- Appearance -->
+      <visual>
+        <origin xyz="0.0 0.0 0.0" rpy="0.0 0.0 0.0" />
+        <geometry>
+          <cylinder radius="${radius}" length="${length}"/>
+        </geometry>
+        <material name="white">
+          <color rgba="1.0 1.0 1.0 0.5"/>
+        </material>
+      </visual>
+    </link>
+  </xacro:macro>
+  <xacro:macro name="imu_link" params="imu_name xyz">
+    <link name="${imu_name}_link">
+      <visual>
+        <origin xyz="0.0 0.0 0.0" rpy="0.0 0.0 0.0" />
+        <geometry>
+          <box size="0.02 0.02 0.02" />
+        </geometry>
+      </visual>
+      <material name="black">
+        <color rgba="0.0 0.0 0.0 0.5"/>
       </material>
-    </visual>
-  </link>
-  <link name="imu_link">
-    <visual>
-      <origin xyz="0.0 0.0 0.0" rpy="0.0 0.0 0.0" />
-      <geometry>
-        <box size="0.02 0.02 0.02" />
-      </geometry>
-    </visual>
-    <material name="black">
-      <color rgba="0.0 0.0 0.0 0.5"/>
-    </material>
-  </link>
-  <joint name="imu_joint" type="fixed">
-    <parent link="base_link" />
-    <child link="imu_link" />
-    <origin xyz="0.0 0.0 0.03" rpy="0.0 0.0 0.0" />
-  </joint>
+    </link>
+    <joint name="${imu_name}_joint" type="fixed">
+      <parent link="base_link" />
+      <child link="${imu_name}_link" />
+      <origin xyz="${xyz}" rpy="0.0 0.0 0.0" />
+    </joint>
+  </xacro:macro>
+  <xacro:base_link radius='0.1' length='0.12' />
+  <xacro:imu_link imu_name="imu_up" xyz="0.0 0.0 0.03" />
+  <xacro:imu_link imu_name="imu_down" xyz="0.0 0.0 -0.03" />
 </robot>
