Commit message: Add base_footprint.

File: chapter6_ws/src/firstbot_description/urdf/fishbot/base.urdf.xacro (robot description, xacro)
@@ -2,6 +2,6 @@
 <robot xmlns:xacro="http://www.ros.org/wiki/xacro">
   <xacro:macro name="base_xacro" params="radius length">
+    <link name="base_footprint" />
     <link name="base_link">
-      <!-- Appearance -->
       <visual>
         <origin xyz="0.0 0.0 0.0" rpy="0.0 0.0 0.0" />
@@ -14,4 +14,9 @@
       </visual>
     </link>
+    <joint name="base_joint" type="fixed">
+      <origin xyz="0.0 0.0 ${length / 2.0 + 0.032 - 0.001}" rpy="0.0 0.0 0.0"/>
+      <parent link="base_footprint"/>
+      <child link="base_link"/>
+    </joint>
   </xacro:macro>
 </robot>
