Commit message: Update fishbot.

File: chapter6_ws/src/firstbot_description/urdf/fishbot/fishbot.urdf.xacro (robot description, xacro)
@@ -6,3 +6,6 @@
   <xacro:include filename="$(find firstbot_description)/urdf/fishbot/sensor/laser.urdf.xacro" />
   <xacro:base_xacro length="0.12" radius="0.1" />
+  <xacro:imu_xacro xyz="0.0 0.0 0.02" />
+  <xacro:camera_xacro xyz="0.1 0.0 0.075" />
+  <xacro:laser_xacro xyz="0.0 0.0 0.1" />
 </robot>

File: chapter6_ws/src/firstbot_description/urdf/fishbot/sensor/camera.urdf.xacro (robot description, xacro)
@@ -6,5 +6,5 @@
         <origin xyz="0.0 0.0 0.0" rpy="0.0 0.0 0.0" />
         <geometry>
-          <box size="0.02 0.02 0.02" />
+          <box size="0.02 0.1 0.02" />
         </geometry>
       </visual>

Commit message: Rename plugin.

File: chapter6_ws/src/firstbot_description/urdf/fishbot/fishbot.urdf.xacro (robot description, xacro)
@@ -7,6 +7,6 @@
   <xacro:include filename="$(find firstbot_description)/urdf/fishbot/actuator/wheel.urdf.xacro" />
   <xacro:include filename="$(find firstbot_description)/urdf/fishbot/actuator/caster.urdf.xacro" />
-  <xacro:include filename="$(find firstbot_description)/urdf/fishbot/plurgins/gazebo_control_plurgin.xacro" />
-  <xacro:include filename="$(find firstbot_description)/urdf/fishbot/plurgins/gazebo_sensor_plurgin.xacro" />
+  <xacro:include filename="$(find firstbot_description)/urdf/fishbot/plugins/gazebo_control_plugin.xacro" />
+  <xacro:include filename="$(find firstbot_description)/urdf/fishbot/plugins/gazebo_sensor_plugin.xacro" />
   <xacro:base_xacro length="0.12" radius="0.1" />
   <xacro:imu_xacro xyz="0.0 0.0 0.02" />
@@ -17,5 +17,5 @@
   <xacro:caster_xacro caster_name="front_caster" xyz="0.08 0.0 -0.076" />
   <xacro:caster_xacro caster_name="back_caster" xyz="-0.08 0.0 -0.076" />
-  <xacro:gazebo_control_plurgin />
-  <xacro:gazebo_sensor_plurgin />
+  <xacro:gazebo_control_plugin />
+  <xacro:gazebo_sensor_plugin />
 </robot>

File: chapter6_ws/src/firstbot_description/urdf/fishbot/plurgins/gazebo_control_plugin.xacro (robot description, xacro)
@@ -1,5 +1,5 @@
 <?xml version="1.0"?>
 <robot xmlns:xacro="http://www.ros.org/wiki/xacro">
-    <xacro:macro name="gazebo_control_plurgin">
+    <xacro:macro name="gazebo_control_plugin">
         <gazebo>
             <plugin name='diff_drive' filename='libgazebo_ros_diff_drive.so'>

File: chapter6_ws/src/firstbot_description/urdf/fishbot/plurgins/gazebo_sensor_plugin.xacro (robot description, xacro)
@@ -1,5 +1,5 @@
 <?xml version="1.0"?>
 <robot xmlns:xacro="http://www.ros.org/wiki/xacro">
-    <xacro:macro name="gazebo_sensor_plurgin">
+    <xacro:macro name="gazebo_sensor_plugin">
         <gazebo reference="laser_link">
             <sensor name="laserscan" type="ray">
