Commit message: Add collision.

File: chapter6_ws/src/firstbot_description/urdf/fishbot/actuator/caster.urdf.xacro (robot description, xacro)
@@ -9,4 +9,10 @@
         </geometry>
       </visual>
+      <collision>
+        <origin xyz="0.0 0.0 0.0" rpy="0 0.0 0.0" />
+        <geometry>
+          <sphere radius="0.016"/>
+        </geometry>
+      </collision>
       <material name="yellow">
         <color rgba="1.0 1.0 0.0 0.8"/>

File: chapter6_ws/src/firstbot_description/urdf/fishbot/actuator/wheel.urdf.xacro (robot description, xacro)
@@ -9,4 +9,10 @@
         </geometry>
       </visual>
+      <collision>
+        <origin xyz="0.0 0.0 0.0" rpy="1.57079 0.0 0.0" />
+        <geometry>
+          <cylinder radius="0.032" length="0.04"/>
+        </geometry>
+      </collision>
       <material name="yellow">
         <color rgba="1.0 1.0 0.0 0.8"/>

File: chapter6_ws/src/firstbot_description/urdf/fishbot/base.urdf.xacro (robot description, xacro)
@@ -13,4 +13,10 @@
         </material>
       </visual>
+      <collision>
+        <origin xyz="0.0 0.0 0.0" rpy="0.0 0.0 0.0" />
+        <geometry>
+          <cylinder radius="${radius}" length="${length}"/>
+        </geometry>
+      </collision>
     </link>
     <joint name="base_joint" type="fixed">

File: chapter6_ws/src/firstbot_description/urdf/fishbot/sensor/camera.urdf.xacro (robot description, xacro)
@@ -9,4 +9,10 @@
         </geometry>
       </visual>
+      <collision>
+        <origin xyz="0.0 0.0 0.0" rpy="0.0 0.0 0.0" />
+        <geometry>
+          <box size="0.02 0.1 0.02" />
+        </geometry>
+      </collision>
       <material name="blue">
         <color rgba="0.0 0.0 1.0 0.5"/>

File: chapter6_ws/src/firstbot_description/urdf/fishbot/sensor/imu.urdf.xacro (robot description, xacro)
@@ -9,4 +9,10 @@
         </geometry>
       </visual>
+      <collision>
+        <origin xyz="0.0 0.0 0.0" rpy="0.0 0.0 0.0" />
+        <geometry>
+          <box size="0.02 0.02 0.02" />
+        </geometry>
+      </collision>
       <material name="black">
         <color rgba="0.0 0.0 0.0 0.5"/>

File: chapter6_ws/src/firstbot_description/urdf/fishbot/sensor/laser.urdf.xacro (robot description, xacro)
@@ -9,4 +9,10 @@
         </geometry>
       </visual>
+      <collision>
+        <origin xyz="0.0 0.0 0.0" rpy="0.0 0.0 0.0" />
+        <geometry>
+          <cylinder radius='0.01' length='0.1' />
+        </geometry>
+      </collision>
       <material name="dark_green">
         <color rgba="0.0 1.0 0.0 0.9"/>
@@ -20,4 +26,10 @@
         </geometry>
       </visual>
+      <collision>
+        <origin xyz="0.0 0.0 0.0" rpy="0.0 0.0 0.0" />
+        <geometry>
+          <cylinder radius='0.02' length='0.02' />
+        </geometry>
+      </collision>
       <material name="light_green">
         <color rgba="0.0 1.0 0.0 0.7"/>
