Commit message: Add gazebo color in xacro.

File: chapter6_ws/src/firstbot_description/urdf/fishbot/sensor/laser.urdf.xacro (robot description, xacro)
@@ -49,4 +49,10 @@
       <origin xyz="${xyz}" rpy="0.0 0.0 0.0" />
     </joint>
+    <gazebo reference="laser_cylinder_link">
+      <material>Gazebo/Black</material>
+    </gazebo>
+    <gazebo reference="laser_link">
+      <material>Gazebo/Black</material>
+    </gazebo>
   </xacro:macro>
 </robot>
