Commit message: Change color.

File: chapter6_ws/src/firstbot_description/urdf/fishbot/sensor/camera.urdf.xacro (robot description, xacro)
@@ -9,6 +9,6 @@
         </geometry>
       </visual>
-      <material name="black">
-        <color rgba="0.0 0.0 0.0 0.5"/>
+      <material name="blue">
+        <color rgba="0.0 0.0 1.0 0.5"/>
       </material>
     </link>

File: chapter6_ws/src/firstbot_description/urdf/fishbot/sensor/laser.urdf.xacro (robot description, xacro)
@@ -9,6 +9,6 @@
         </geometry>
       </visual>
-      <material name="black">
-        <color rgba="0.0 0.0 0.0 1.0"/>
+      <material name="dark_green">
+        <color rgba="0.0 1.0 0.0 0.9"/>
       </material>
     </link>
@@ -20,6 +20,6 @@
         </geometry>
       </visual>
-      <material name="black">
-        <color rgba="0.0 0.0 0.0 1.0"/>
+      <material name="light_green">
+        <color rgba="0.0 1.0 0.0 0.7"/>
       </material>
     </link>

Commit message: Add camera_optical_joint.

File: chapter6_ws/src/firstbot_description/urdf/fishbot/sensor/camera.urdf.xacro (robot description, xacro)
@@ -21,4 +21,5 @@
       <xacro:box_inertia m="0.05" w="0.02" h="0.1" d="0.02" />
     </link>
+    <link name="camera_optical_link" />
     <joint name="camera_joint" type="fixed">
       <parent link="base_link" />
@@ -26,4 +27,9 @@
       <origin xyz="${xyz}" rpy="0.0 0.0 0.0" />
     </joint>
+    <joint name="camera_optical_joint" type="fixed">
+      <parent link="camera_link" />
+      <child link="camera_optical_link" />
+      <origin xyz="0 0 0" rpy="${-pi/2} 0.0 ${-pi/2}" />
+    </joint>
   </xacro:macro>
 </robot>
