Commit message: Add base_footprint.

File: fishbot/ws/urdf/base.urdf.xacro (robot description, xacro)
@@ -2,4 +2,5 @@
 <robot xmlns:xacro="http://www.ros.org/wiki/xacro">
   <xacro:macro name="base_xacro" params="radius length">
+    <link name="base_footprint" />
     <link name="base_link">
       <visual>
@@ -12,5 +13,19 @@
         </material>
       </visual>
+      <collision>
+        <origin xyz="0.0 0.0 0.0" rpy="0.0 0.0 0.0" />
+        <geometry>
+          <cylinder radius="${radius}" length="${length}"/>
+        </geometry>
+        <material name="white">
+          <color rgba="1.0 1.0 1.0 0.5"/>
+        </material>
+      </collision>
     </link>
+    <joint name="base_joint" type="fixed">
+      <parent link="base_footprint" />
+      <child link="base_link" />
+      <origin xyz="0 0 ${length/2.0 + 0.032 - 0.001}" rpy="0 0 0" />
+    </joint>
   </xacro:macro>
 </robot>
