Commit message: Add diff_drive.

File: fishbot/ws/urdf/actuator/wheel.urdf.xacro (robot description, xacro)
@@ -3,5 +3,5 @@
   <xacro:include filename="$(find fishbot)/urdf/common_inertia.xacro" />
   <xacro:macro name="wheel_xacro" params="wheel_name xyz">
-    <link name="${wheel_name}_link">
+    <link name="${wheel_name}_wheel_link">
       <visual>
         <origin xyz="0.0 0.0 0.0" rpy="1.57079 0.0 0.0" />
@@ -21,11 +21,11 @@
       <xacro:cylinder_inertia m="0.05" r="0.032" h="0.04" />
     </link>
-    <joint name="${wheel_name}_joint" type="continuous">
+    <joint name="${wheel_name}_wheel_joint" type="continuous">
       <parent link="base_link" />
-      <child link="${wheel_name}_link" />
+      <child link="${wheel_name}_wheel_link" />
       <origin xyz="${xyz}" rpy="0.0 0.0 0.0" />
       <axis xyz="0.0 1 0.0"/>
     </joint>
-    <gazebo reference="${wheel_name}_link">
+    <gazebo reference="${wheel_name}_wheel_link">
       <material>Gazebo/Black</material>
       <mu1 value="20.0" />

File: fishbot/ws/urdf/fishbot.urdf.xacro (robot description, xacro)
@@ -7,4 +7,5 @@
   <xacro:include filename="$(find fishbot)/urdf/actuator/wheel.urdf.xacro" />
   <xacro:include filename="$(find fishbot)/urdf/actuator/caster.urdf.xacro" />
+  <xacro:include filename="$(find fishbot)/urdf/plugins/gazebo_control_plugin.xacro" />
   <xacro:base_xacro length="0.12" radius="0.1" />
   <xacro:imu_xacro xyz="0.0 0.0 0.02" />
@@ -15,3 +16,4 @@
   <xacro:caster_xacro caster_name="front" xyz="0.08 0 -0.076" />
   <xacro:caster_xacro caster_name="back" xyz="-0.08 0 -0.076" />
+  <xacro:gazebo_control_plugin />
 </robot>
