Commit message: Add collision.

File: fishbot/ws/urdf/actuator/caster.urdf.xacro (robot description, xacro)
@@ -9,4 +9,10 @@
         </geometry>
       </visual>
+      <collision>
+        <origin xyz="0 0 0" rpy="0 0 0" />
+        <geometry>
+          <sphere radius="0.016"/>
+        </geometry>
+      </collision>
       <material name="yellow">
         <color rgba="1.0 1.0 0.0 0.8"/>

File: fishbot/ws/urdf/actuator/wheel.urdf.xacro (robot description, xacro)
@@ -9,4 +9,10 @@
         </geometry>
       </visual>
+      <collision>
+        <origin xyz="0.0 0.0 0.0" rpy="1.57079 0.0 0.0" />
+        <geometry>
+          <cylinder radius="0.032" length="0.04"/>
+        </geometry>
+      </collision>
       <material name="yellow">
         <color rgba="1.0 1.0 0.0 0.8"/>

File: fishbot/ws/urdf/sensor/camera.urdf.xacro (robot description, xacro)
@@ -9,4 +9,10 @@
         </geometry>
       </visual>
+      <collision>
+        <origin xyz="0.0 0.0 0.0" rpy="0.0 0.0 0.0" />
+        <geometry>
+          <box size="0.02 0.1 0.02" />
+        </geometry>
+      </collision>
       <material name="blue">
         <color rgba="0.0 0.0 1.0 0.5"/>

File: fishbot/ws/urdf/sensor/imu.urdf.xacro (robot description, xacro)
@@ -9,4 +9,10 @@
         </geometry>
       </visual>
+      <collision>
+        <origin xyz="0.0 0.0 0.0" rpy="0.0 0.0 0.0" />
+        <geometry>
+          <box size="0.02 0.02 0.02" />
+        </geometry>
+      </collision>
       <material name="black">
         <color rgba="0.0 0.0 0.0 0.5"/>

File: fishbot/ws/urdf/sensor/laser.urdf.xacro (robot description, xacro)
@@ -9,4 +9,10 @@
         </geometry>
       </visual>
+      <collision>
+        <origin xyz="0.0 0.0 0.0" rpy="0.0 0.0 0.0" />
+        <geometry>
+          <cylinder radius='0.01' length='0.1' />
+        </geometry>
+      </collision>
       <material name="dark_green">
         <color rgba="0.0 1.0 0.0 0.9"/>
@@ -20,4 +26,10 @@
         </geometry>
       </visual>
+      <collision>
+        <origin xyz="0.0 0.0 0.0" rpy="0.0 0.0 0.0" />
+        <geometry>
+          <cylinder radius='0.02' length='0.02' />
+        </geometry>
+      </collision>
       <material name="light_green">
         <color rgba="0.0 1.0 0.0 0.7"/>

Commit message: Set color in gazebo.

File: fishbot/ws/urdf/actuator/caster.urdf.xacro (robot description, xacro)
@@ -27,4 +27,7 @@
       <axis xyz="0 0 0"/>
     </joint>
+    <gazebo reference="${caster_name}_link">
+      <material>Gazebo/DarkGrey</material>
+    </gazebo>
   </xacro:macro>
 </robot>

File: fishbot/ws/urdf/actuator/wheel.urdf.xacro (robot description, xacro)
@@ -27,4 +27,7 @@
       <axis xyz="0.0 1 0.0"/>
     </joint>
+    <gazebo reference="${wheel_name}_link">
+      <material>Gazebo/Black</material>
+    </gazebo>
   </xacro:macro>
 </robot>

File: fishbot/ws/urdf/base.urdf.xacro (robot description, xacro)
@@ -30,4 +30,7 @@
       <origin xyz="0 0 ${length/2.0 + 0.032 - 0.001}" rpy="0 0 0" />
     </joint>
+    <gazebo reference="base_link">
+      <material>Gazebo/SkyBlue</material>
+    </gazebo>
   </xacro:macro>
 </robot>

File: fishbot/ws/urdf/sensor/camera.urdf.xacro (robot description, xacro)
@@ -26,4 +26,7 @@
       <origin xyz="${xyz}" rpy="0.0 0.0 0.0" />
     </joint>
+    <gazebo reference="camera_link">
+      <material>Gazebo/Red</material>
+    </gazebo>
   </xacro:macro>
 </robot>

File: fishbot/ws/urdf/sensor/laser.urdf.xacro (robot description, xacro)
@@ -49,4 +49,10 @@
       <origin xyz="0.0 0.0 0.05" rpy="0.0 0.0 0.0" />
     </joint>
+    <gazebo reference="laser_cylinder_link">
+      <material>Gazebo/DarkGrey</material>
+    </gazebo>
+    <gazebo reference="laser_link">
+      <material>Gazebo/Orange</material>
+    </gazebo>
   </xacro:macro>
 </robot>

Commit message: Update caster name.

File: fishbot/ws/urdf/actuator/caster.urdf.xacro (robot description, xacro)
@@ -3,5 +3,5 @@
   <xacro:include filename="$(find fishbot)/urdf/common_inertia.xacro" />
   <xacro:macro name="caster_xacro" params="caster_name xyz">
-    <link name="${caster_name}_link">
+    <link name="${caster_name}_caster_link">
       <visual>
         <origin xyz="0 0 0" rpy="0 0 0" />
@@ -23,9 +23,9 @@
     <joint name="${caster_name}_joint" type="fixed">
       <parent link="base_link" />
-      <child link="${caster_name}_link" />
+      <child link="${caster_name}_caster_link" />
       <origin xyz="${xyz}" rpy="0 0 0" />
       <axis xyz="0 0 0"/>
     </joint>
-    <gazebo reference="${caster_name}_link">
+    <gazebo reference="${caster_name}_caster_link">
       <material>Gazebo/DarkGrey</material>
       <mu1 value="0.0" />
