Commit message: Add camera_optical_link.

File: fishbot/ws/urdf/sensor/camera.urdf.xacro (robot description, xacro)
@@ -21,8 +21,14 @@
       <xacro:box_inertia m="0.05" w="0.02" h="0.1" d="0.02" />
     </link>
+    <link name="camera_optical_link" />
     <joint name="camera_joint" type="fixed">
       <parent link="base_link" />
       <child link="camera_link" />
       <origin xyz="${xyz}" rpy="0.0 0.0 0.0" />
+    </joint>
+    <joint name="camera_optical_joint" type="fixed">
+      <parent link="camera_link" />
+      <child link="camera_optical_link" />
+      <origin xyz="0 0 0" rpy="${-pi/2} 0.0 ${-pi/2}" />
     </joint>
     <gazebo reference="camera_link">
